File: Prototype-PCB/Prototype-PCB.sch (KiCad schematic (older format))
At the start: 9 parts, among them SW1 SW_SPST, SW2 SW_SPST, SW3 SW_SPST, SW4 SW_SPST

Commit message: Made pcb prototype with vias connecting SMD components on both sides.
Parts:
- R1, RTRACK1: footprint (none) -> 3Meg SMT Resistor:KTR18EZPF3004
- R2: footprint (none) -> 2Meg SMT Resistor:KTR18EZPF2004
- R3: footprint (none) -> 1Meg SMT Resistor:KTR18EZPF1004
- R4: footprint (none) -> 750k SMT Resistor:KTR18EZPF7503
- SW1, SW2, SW3, SW4: footprint (none) -> KSR221GNCLFS-SMT:KSR221GNCLFS-SMT-NCSPST
Changed lines of the file:
@@
 EESchema Schematic File Version 4
+LIBS:Prototype-PCB-cache
 EELAYER 29 0
 EELAYER END
@@
 F 0 "SW1" H 4500 3785 50  0000 C CNN
 F 1 "SW_SPST" H 4500 3694 50  0000 C CNN
-F 2 "" H 4500 3550 50  0001 C CNN
+F 2 "KSR221GNCLFS-SMT:KSR221GNCLFS-SMT-NCSPST" H 4500 3550 50  0001 C CNN
 F 3 "~" H 4500 3550 50  0001 C CNN
 	1    4500 3550
@@
 F 0 "RTRACK1" V 3695 3550 50  0000 C CNN
 F 1 "3Meg" V 3786 3550 50  0000 C CNN
-F 2 "" H 3900 3550 50  0001 C CNN
+F 2 "3Meg SMT Resistor:KTR18EZPF3004" H 3900 3550 50  0001 C CNN
 F 3 "~" H 3900 3550 50  0001 C CNN
 	1    3900 3550
@@
 F 0 "R1" V 4295 3950 50  0000 C CNN
 F 1 "3Meg" V 4386 3950 50  0000 C CNN
-F 2 "" H 4500 3950 50  0001 C CNN
+F 2 "3Meg SMT Resistor:KTR18EZPF3004" H 4500 3950 50  0001 C CNN
 F 3 "~" H 4500 3950 50  0001 C CNN
 	1    4500 3950
@@
 F 0 "SW2" H 5300 3785 50  0000 C CNN
 F 1 "SW_SPST" H 5300 3694 50  0000 C CNN
-F 2 "" H 5300 3550 50  0001 C CNN
+F 2 "KSR221GNCLFS-SMT:KSR221GNCLFS-SMT-NCSPST" H 5300 3550 50  0001 C CNN
 F 3 "~" H 5300 3550 50  0001 C CNN
 	1    5300 3550
@@
 F 0 "R2" V 5095 3950 50  0000 C CNN
 F 1 "2Meg" V 5186 3950 50  0000 C CNN
-F 2 "" H 5300 3950 50  0001 C CNN
+F 2 "2Meg SMT Resistor:KTR18EZPF2004" H 5300 3950 50  0001 C CNN
 F 3 "~" H 5300 3950 50  0001 C CNN
 	1    5300 3950
@@
 F 0 "SW3" H 6050 3785 50  0000 C CNN
 F 1 "SW_SPST" H 6050 3694 50  0000 C CNN
-F 2 "" H 6050 3550 50  0001 C CNN
+F 2 "KSR221GNCLFS-SMT:KSR221GNCLFS-SMT-NCSPST" H 6050 3550 50  0001 C CNN
 F 3 "~" H 6050 3550 50  0001 C CNN
 	1    6050 3550
@@
 F 0 "R3" V 5845 3950 50  0000 C CNN
 F 1 "1Meg" V 5936 3950 50  0000 C CNN
-F 2 "" H 6050 3950 50  0001 C CNN
+F 2 "1Meg SMT Resistor:KTR18EZPF1004" H 6050 3950 50  0001 C CNN
 F 3 "~" H 6050 3950 50  0001 C CNN
 	1    6050 3950
@@
 F 0 "SW4" H 6850 3785 50  0000 C CNN
 F 1 "SW_SPST" H 6850 3694 50  0000 C CNN
-F 2 "" H 6850 3550 50  0001 C CNN
+F 2 "KSR221GNCLFS-SMT:KSR221GNCLFS-SMT-NCSPST" H 6850 3550 50  0001 C CNN
 F 3 "~" H 6850 3550 50  0001 C CNN
 	1    6850 3550
@@
 F 0 "R4" V 6645 3950 50  0000 C CNN
 F 1 "750k" V 6736 3950 50  0000 C CNN
-F 2 "" H 6850 3950 50  0001 C CNN
+F 2 "750k SMT Resistor:KTR18EZPF7503" H 6850 3950 50  0001 C CNN
 F 3 "~" H 6850 3950 50  0001 C CNN
 	1    6850 3950
