File: Prototype-PCB/Prototype-PCB.sch (KiCad schematic (older format))
At the start: 9 parts, among them SW1 SW_SPST, SW2 SW_SPST, SW3 SW_SPST, SW4 SW_SPST

Commit message: Modified the pcb file. Changed the footprints for SMT resistors.
Parts:
- R1, RTRACK1: footprint 3Meg SMT Resistor:KTR18EZPF3004 -> Read-Rope:R_1206_3216Metric_Pad1.42x1.75mm_HandSolder
- R2: footprint 2Meg SMT Resistor:KTR18EZPF2004 -> Read-Rope:R_1206_3216Metric_Pad1.42x1.75mm_HandSolder
- R3: footprint 1Meg SMT Resistor:KTR18EZPF1004 -> Read-Rope:R_1206_3216Metric_Pad1.42x1.75mm_HandSolder
- R4: footprint 750k SMT Resistor:KTR18EZPF7503 -> Read-Rope:R_1206_3216Metric_Pad1.42x1.75mm_HandSolder
- SW1, SW2, SW3, SW4: footprint KSR221GNCLFS-SMT:KSR221GNCLFS-SMT-NCSPST -> Read-Rope:KSR221GNCLFS-SMT-NCSPST
Changed lines of the file:
@@
 F 0 "SW1" H 4500 3785 50  0000 C CNN
 F 1 "SW_SPST" H 4500 3694 50  0000 C CNN
-F 2 "KSR221GNCLFS-SMT:KSR221GNCLFS-SMT-NCSPST" H 4500 3550 50  0001 C CNN
+F 2 "Read-Rope:KSR221GNCLFS-SMT-NCSPST" H 4500 3550 50  0001 C CNN
 F 3 "~" H 4500 3550 50  0001 C CNN
 	1    4500 3550
@@
 F 0 "RTRACK1" V 3695 3550 50  0000 C CNN
 F 1 "20k" V 3786 3550 50  0000 C CNN
-F 2 "3Meg SMT Resistor:KTR18EZPF3004" H 3900 3550 50  0001 C CNN
+F 2 "Read-Rope:R_1206_3216Metric_Pad1.42x1.75mm_HandSolder" H 3900 3550 50  0001 C CNN
 F 3 "~" H 3900 3550 50  0001 C CNN
 	1    3900 3550
@@
 F 0 "R1" V 4295 3950 50  0000 C CNN
 F 1 "9k" V 4386 3950 50  0000 C CNN
-F 2 "3Meg SMT Resistor:KTR18EZPF3004" H 4500 3950 50  0001 C CNN
+F 2 "Read-Rope:R_1206_3216Metric_Pad1.42x1.75mm_HandSolder" H 4500 3950 50  0001 C CNN
 F 3 "~" H 4500 3950 50  0001 C CNN
 	1    4500 3950
@@
 F 0 "SW2" H 5300 3785 50  0000 C CNN
 F 1 "SW_SPST" H 5300 3694 50  0000 C CNN
-F 2 "KSR221GNCLFS-SMT:KSR221GNCLFS-SMT-NCSPST" H 5300 3550 50  0001 C CNN
+F 2 "Read-Rope:KSR221GNCLFS-SMT-NCSPST" H 5300 3550 50  0001 C CNN
 F 3 "~" H 5300 3550 50  0001 C CNN
 	1    5300 3550
@@
 F 0 "R2" V 5095 3950 50  0000 C CNN
 F 1 "7k" V 5186 3950 50  0000 C CNN
-F 2 "2Meg SMT Resistor:KTR18EZPF2004" H 5300 3950 50  0001 C CNN
+F 2 "Read-Rope:R_1206_3216Metric_Pad1.42x1.75mm_HandSolder" H 5300 3950 50  0001 C CNN
 F 3 "~" H 5300 3950 50  0001 C CNN
 	1    5300 3950
@@
 F 0 "SW3" H 6050 3785 50  0000 C CNN
 F 1 "SW_SPST" H 6050 3694 50  0000 C CNN
-F 2 "KSR221GNCLFS-SMT:KSR221GNCLFS-SMT-NCSPST" H 6050 3550 50  0001 C CNN
+F 2 "Read-Rope:KSR221GNCLFS-SMT-NCSPST" H 6050 3550 50  0001 C CNN
 F 3 "~" H 6050 3550 50  0001 C CNN
 	1    6050 3550
@@
 F 0 "R3" V 5845 3950 50  0000 C CNN
 F 1 "3k" V 5936 3950 50  0000 C CNN
-F 2 "1Meg SMT Resistor:KTR18EZPF1004" H 6050 3950 50  0001 C CNN
+F 2 "Read-Rope:R_1206_3216Metric_Pad1.42x1.75mm_HandSolder" H 6050 3950 50  0001 C CNN
 F 3 "~" H 6050 3950 50  0001 C CNN
 	1    6050 3950
@@
 F 0 "SW4" H 6850 3785 50  0000 C CNN
 F 1 "SW_SPST" H 6850 3694 50  0000 C CNN
-F 2 "KSR221GNCLFS-SMT:KSR221GNCLFS-SMT-NCSPST" H 6850 3550 50  0001 C CNN
+F 2 "Read-Rope:KSR221GNCLFS-SMT-NCSPST" H 6850 3550 50  0001 C CNN
 F 3 "~" H 6850 3550 50  0001 C CNN
 	1    6850 3550
@@
 F 0 "R4" V 6645 3950 50  0000 C CNN
 F 1 "1k" V 6736 3950 50  0000 C CNN
-F 2 "750k SMT Resistor:KTR18EZPF7503" H 6850 3950 50  0001 C CNN
+F 2 "Read-Rope:R_1206_3216Metric_Pad1.42x1.75mm_HandSolder" H 6850 3950 50  0001 C CNN
 F 3 "~" H 6850 3950 50  0001 C CNN
 	1    6850 3950
